Commit message: Added laser to gazebo urdf

File: corobot_description/urdf/corobot.urdf.xacro (robot description, xacro)
@@ -105,5 +105,5 @@
     <xacro:plate name="first_plate" length="0.310" width="0.280"/>
     <xacro:plate name="top_plate" length="0.217" width="0.280"/>
-    <link name="laser">
+    <link name="laser_link">
         <visual>
             <geometry>
@@ -130,5 +130,5 @@
     <joint name="laser_joint" type="fixed">
         <parent link="first_plate"/>
-        <child link="laser"/>
+        <child link="laser_link"/>
         <origin xyz="0.135 -0.075 -0.035" rpy="${pi} 0 0"/>
     </joint>

Commit message: Tweaked robot description

File: corobot_description/urdf/corobot.urdf.xacro (robot description, xacro)
@@ -5,5 +5,5 @@
     <xacro:property name="BASE_WIDTH" value="0.201" />
     <xacro:property name="BASE_HEIGHT" value="0.060" />
-    <xacro:property name="BASE_MASS" value="1.0" />
+    <xacro:property name="BASE_MASS" value="8.6" />
     <xacro:property name="WHEEL_THICKNESS" value="0.065" />
     <xacro:property name="WHEEL_RADIUS" value="0.060" />
@@ -11,5 +11,5 @@
     <xacro:property name="WHEELBASE" value="0.280" />
     <xacro:property name="AXLE_AXLE" value="0.190" />
-    <xacro:property name="WHEEL_MASS" value="0.1" />
+    <xacro:property name="WHEEL_MASS" value="0.9" />
     <xacro:property name="WHEEL_MOMENT" value="${WHEEL_MASS/12*(3*WHEEL_RADIUS**2+WHEEL_THICKNESS**2)}" />
     <xacro:property name="PLATE_THICKNESS" value="0.006"/>
@@ -43,5 +43,5 @@
                 </geometry>
             </collision>
-            <xacro:box_inertia x="${length}" y="${width}" z="${PLATE_THICKNESS}" mass="0"/>
+            <xacro:box_inertia x="${length}" y="${width}" z="${PLATE_THICKNESS}" mass="0.1"/>
         </link>
     </xacro:macro>
@@ -82,5 +82,10 @@
         </transmission>
     </xacro:macro>
-    <link name="base_link">
+    <link name="base_link"/>
+    <joint name="base_joint" type="fixed">
+        <parent link="base_link"/>
+        <child link="base"/>
+    </joint>
+    <link name="base">
         <visual>
             <geometry>
@@ -94,12 +99,5 @@
             </geometry>
         </collision>
-        <inertial>
-            <mass value="${BASE_MASS}"/>
-            <inertia
-                ixx="${BASE_MASS/12*(BASE_HEIGHT**2+BASE_LENGTH**2)}"
-                iyy="${BASE_MASS/12*(BASE_WIDTH**2+BASE_LENGTH**2)}"
-                izz="${BASE_MASS/12*(BASE_WIDTH**2+BASE_HEIGHT**2)}"
-                ixy="0" ixz="0" iyz="0"/>
-        </inertial>
+        <box_inertia x="${BASE_LENGTH}" y="${BASE_WIDTH}" z="${BASE_HEIGHT}" mass="${BASE_MASS}"/>
     </link>
     <xacro:plate name="first_plate" length="0.310" width="0.280"/>
